Commit message: merged build and controller manager test

File: src/robot_description/urdf/robot.urdf.xacro (robot description, xacro)
@@ -3,15 +3,15 @@
   <!-- === PROPERTIES === -->
   <!-- Wheels -->
-  <xacro:property name="wheel_radius"   value="0.0325"/>            <!-- 6.5 cm / 2 -->
-  <xacro:property name="wheel_separation" value="0.29"/>            <!-- 29 cm -->
-  <xacro:property name="wheel_width"    value="0.024"/>             <!-- 2.4 cm -->
-  <xacro:property name="wheel_mass"     value="0.10"/>              <!-- approx. 100 g -->
+  <xacro:property name="wheel_radius"       value="0.0325"/>            <!-- 6.5 cm / 2 -->
+  <xacro:property name="wheel_separation"   value="0.29"/>              <!-- 29 cm -->
+  <xacro:property name="wheel_width"        value="0.024"/>             <!-- 2.4 cm -->
+  <xacro:property name="wheel_mass"         value="0.10"/>              <!-- approx. 100 g -->
   <!-- I = ½ m r² for a solid cylinder -->
-  <xacro:property name="wheel_inertia"  value="${0.5 * wheel_mass * wheel_radius * wheel_radius}"/>
+  <xacro:property name="wheel_inertia"      value="${0.5 * wheel_mass * wheel_radius * wheel_radius}"/>
   <!-- Base (chassis) -->
-  <xacro:property name="base_mass"      value="${15 * 0.45359237}"/> <!-- 15 lbs → kg -->
-  <xacro:property name="base_length"    value="0.37"/>             <!-- 37 cm -->
-  <xacro:property name="base_width"     value="0.42"/>             <!-- 42 cm -->
-  <xacro:property name="base_height"    value="0.60"/>             <!-- 60 cm -->
+  <xacro:property name="base_mass"          value="${15 * 0.45359237}"/> <!-- 15 lbs → kg -->
+  <xacro:property name="base_length"        value="0.37"/>              <!-- 37 cm -->
+  <xacro:property name="base_width"         value="0.42"/>              <!-- 42 cm -->
+  <xacro:property name="base_height"        value="0.60"/>              <!-- 60 cm -->
   <!-- Rectangular prism inertia -->
   <xacro:property name="ixx" value="${base_mass * (base_width*base_width + base_height*base_height) / 12.0}"/>
@@ -19,21 +19,17 @@
   <xacro:property name="izz" value="${base_mass * (base_length*base_length + base_width*base_width)  / 12.0}"/>
   <!-- IMU -->
-  <!-- placed at (0,0) in XY and 2 cm above axle (wheel_radius + 0.02) in Z -->
   <xacro:property name="imu_xyz"  value="0 0 ${wheel_radius + 0.02}"/>
-  <!-- yaw 180° so X-axis of IMU faces rear -->
   <xacro:property name="imu_rpy"  value="0 0 3.14159"/>
   <!-- LiDAR -->
-  <!-- centered in XY, 60 cm above axles -->
   <xacro:property name="lidar_xyz" value="0 0 ${wheel_radius + 0.60}"/>
   <xacro:property name="lidar_rpy" value="0 0 0"/>
   <!-- Camera -->
-  <!-- centered in Y, 15 cm forward (+X), 55 cm above axles -->
-  <xacro:property name="camera_xyz" value="${0.15} 0 ${wheel_radius + 0.55}"/>
+  <xacro:property name="camera_xyz" value="0.15 0 ${wheel_radius + 0.55}"/>
   <xacro:property name="camera_rpy" value="0 0 0"/>
   <!-- === LINKS & JOINTS === -->
   <link name="base_link">
     <inertial>
-      <mass     value="${base_mass}"/>
-      <origin   xyz="0 0 0" rpy="0 0 0"/>
+      <mass   value="${base_mass}"/>
+      <origin xyz="0 0 0" rpy="0 0 0"/>
       <inertia ixx="${ixx}" ixy="0.0" ixz="0.0"
                iyy="${iyy}" iyz="0.0"
@@ -81,9 +77,9 @@
   <ros2_control name="diffbot_system" type="system">
     <hardware>
+      <!-- plugin stays the same -->
       <plugin>diffbot_hardware/DiffBotSystem</plugin>
-<hardware_parameters>
-  <serial_port>/dev/ttyACM0</serial_port>
-  <baud_rate>115200</baud_rate>
-</hardware_parameters>
+      <!-- these two lines replace your hardware_parameters block -->
+      <param name="serial_port">/dev/ttyACM0</param>
+      <param name="baud_rate">115200</param>
     </hardware>
     <joint name="wheel_left_joint">

Commit message: updated with Elsa's dims

File: src/robot_description/urdf/robot.urdf.xacro (robot description, xacro)
@@ -1,34 +1,39 @@
 <?xml version="1.0"?>
 <robot xmlns:xacro="http://www.ros.org/wiki/xacro" name="diffbot">
+  <!-- === MATERIALS === -->
+  <material name="Green">
+    <color rgba="0 0.6 0 1"/>
+  </material>
+  <material name="Grey">
+    <color rgba="0.7 0.7 0.7 1"/>
+  </material>
+  <material name="White">
+    <color rgba="1 1 1 1"/>
+  </material>
   <!-- === PROPERTIES === -->
   <!-- Wheels -->
-  <xacro:property name="wheel_radius"       value="0.0325"/>            <!-- 6.5 cm / 2 -->
-  <xacro:property name="wheel_separation"   value="0.29"/>              <!-- 29 cm -->
-  <xacro:property name="wheel_width"        value="0.024"/>             <!-- 2.4 cm -->
-  <xacro:property name="wheel_mass"         value="0.10"/>              <!-- approx. 100 g -->
-  <!-- I = ½ m r² for a solid cylinder -->
+  <xacro:property name="wheel_radius"       value="0.0325"/>
+  <xacro:property name="wheel_separation"   value="0.25"/>
+  <xacro:property name="wheel_width"        value="0.027"/>
+  <xacro:property name="wheel_mass"         value="0.034"/>
   <xacro:property name="wheel_inertia"      value="${0.5 * wheel_mass * wheel_radius * wheel_radius}"/>
-  <!-- Base (chassis) -->
-  <xacro:property name="base_mass"          value="${15 * 0.45359237}"/> <!-- 15 lbs → kg -->
-  <xacro:property name="base_length"        value="0.37"/>              <!-- 37 cm -->
-  <xacro:property name="base_width"         value="0.42"/>              <!-- 42 cm -->
-  <xacro:property name="base_height"        value="0.60"/>              <!-- 60 cm -->
-  <!-- Rectangular prism inertia -->
-  <xacro:property name="ixx" value="${base_mass * (base_width*base_width + base_height*base_height) / 12.0}"/>
-  <xacro:property name="iyy" value="${base_mass * (base_length*base_length + base_height*base_height) / 12.0}"/>
-  <xacro:property name="izz" value="${base_mass * (base_length*base_length + base_width*base_width)  / 12.0}"/>
-  <!-- IMU -->
-  <xacro:property name="imu_xyz"  value="0 0 ${wheel_radius + 0.02}"/>
-  <xacro:property name="imu_rpy"  value="0 0 3.14159"/>
-  <!-- LiDAR -->
-  <xacro:property name="lidar_xyz" value="0 0 ${wheel_radius + 0.60}"/>
-  <xacro:property name="lidar_rpy" value="0 0 0"/>
-  <!-- Camera -->
-  <xacro:property name="camera_xyz" value="0.15 0 ${wheel_radius + 0.55}"/>
+  <!-- Base (cylinder chassis) -->
+  <xacro:property name="base_mass"          value="${15 * 0.45359237}"/>
+  <xacro:property name="base_radius"        value="0.21"/>
+  <xacro:property name="base_height"        value="0.55"/>
+  <xacro:property name="ixx" value="${base_mass * (3 * base_radius * base_radius + base_height * base_height) / 12.0}"/>
+  <xacro:property name="iyy" value="${base_mass * (3 * base_radius * base_radius + base_height * base_height) / 12.0}"/>
+  <xacro:property name="izz" value="${0.5 * base_mass * base_radius * base_radius}"/>
+  <!-- Sensors -->
+  <xacro:property name="imu_xyz"    value="0 0 ${wheel_radius + 0.01}"/>
+  <xacro:property name="imu_rpy"    value="0 0 3.14159"/>
+  <xacro:property name="lidar_xyz"  value="0 0 ${wheel_radius + 0.55}"/>
+  <xacro:property name="lidar_rpy"  value="0 0 0"/>
+  <xacro:property name="camera_xyz" value="0.15 0 ${wheel_radius + 0.5}"/>
   <xacro:property name="camera_rpy" value="0 0 0"/>
-  <!-- === LINKS & JOINTS === -->
+  <!-- === LINKS === -->
   <link name="base_link">
     <inertial>
-      <mass   value="${base_mass}"/>
+      <mass value="${base_mass}"/>
       <origin xyz="0 0 0" rpy="0 0 0"/>
       <inertia ixx="${ixx}" ixy="0.0" ixz="0.0"
@@ -36,23 +41,70 @@
                izz="${izz}"/>
     </inertial>
+    <visual>
+      <geometry>
+        <cylinder radius="${base_radius}" length="${base_height}"/>
+      </geometry>
+      <origin xyz="0 0 0" rpy="0 0 0"/>
+      <material name="Green"/>
+    </visual>
   </link>
-  <!-- Left wheel -->
-  <link name="wheel_left_link"/>
+  <link name="wheel_left_link">
+    <visual>
+      <geometry>
+        <cylinder radius="${wheel_radius}" length="${wheel_width}"/>
+      </geometry>
+      <origin xyz="0 0 0" rpy="1.5707 0 0"/>
+      <material name="Grey"/>
+    </visual>
+  </link>
+  <link name="wheel_right_link">
+    <visual>
+      <geometry>
+        <cylinder radius="${wheel_radius}" length="${wheel_width}"/>
+      </geometry>
+      <origin xyz="0 0 0" rpy="1.5707 0 0"/>
+      <material name="Grey"/>
+    </visual>
+  </link>
+  <link name="imu_link">
+    <visual>
+      <geometry>
+        <box size="0.05 0.05 0.02"/>
+      </geometry>
+      <origin xyz="0 0 0" rpy="0 0 0"/>
+      <material name="White"/>
+    </visual>
+  </link>
+  <link name="lidar_link">
+    <visual>
+      <geometry>
+        <cylinder radius="0.05" length="0.03"/>
+      </geometry>
+      <origin xyz="0 0 0" rpy="0 0 0"/>
+      <material name="White"/>
+    </visual>
+  </link>
+  <link name="camera_link">
+    <visual>
+      <geometry>
+        <box size="0.05 0.05 0.05"/>
+      </geometry>
+      <origin xyz="0 0 0" rpy="0 0 0"/>
+      <material name="White"/>
+    </visual>
+  </link>
+  <!-- === JOINTS === -->
   <joint name="wheel_left_joint" type="continuous">
     <parent link="base_link"/>
     <child  link="wheel_left_link"/>
     <origin xyz="0 ${-wheel_separation/2.0} 0" rpy="0 0 0"/>
-    <axis   xyz="0 0 1"/>
+    <axis xyz="0 1 0"/>
   </joint>
-  <!-- Right wheel -->
-  <link name="wheel_right_link"/>
   <joint name="wheel_right_joint" type="continuous">
     <parent link="base_link"/>
     <child  link="wheel_right_link"/>
-    <origin xyz="0 ${ wheel_separation/2.0} 0" rpy="0 0 0"/>
-    <axis   xyz="0 0 1"/>
+    <origin xyz="0 ${wheel_separation/2.0} 0" rpy="0 0 0"/>
+    <axis xyz="0 1 0"/>
   </joint>
-  <!-- IMU mount -->
-  <link name="imu_link"/>
   <joint name="imu_joint" type="fixed">
     <parent link="base_link"/>
@@ -60,6 +112,4 @@
     <origin xyz="${imu_xyz}" rpy="${imu_rpy}"/>
   </joint>
-  <!-- LiDAR mount -->
-  <link name="lidar_link"/>
   <joint name="lidar_joint" type="fixed">
     <parent link="base_link"/>
@@ -67,6 +117,4 @@
     <origin xyz="${lidar_xyz}" rpy="${lidar_rpy}"/>
   </joint>
-  <!-- Camera mount -->
-  <link name="camera_link"/>
   <joint name="camera_joint" type="fixed">
     <parent link="base_link"/>
@@ -77,7 +125,5 @@
   <ros2_control name="diffbot_system" type="system">
     <hardware>
-      <!-- plugin stays the same -->
       <plugin>diffbot_hardware/DiffBotSystem</plugin>
-      <!-- these two lines replace your hardware_parameters block -->
       <param name="serial_port">/dev/ttyACM0</param>
       <param name="baud_rate">115200</param>

Commit message: Modified xacro value and created backup of src

File: src/robot_description/urdf/robot.urdf.xacro (robot description, xacro)
@@ -14,5 +14,5 @@
   <!-- Wheels -->
   <xacro:property name="wheel_radius"       value="0.0325"/>
-  <xacro:property name="wheel_separation"   value="0.25"/>
+  <xacro:property name="wheel_separation"   value="0.292"/>
   <xacro:property name="wheel_width"        value="0.027"/>
   <xacro:property name="wheel_mass"         value="0.034"/>

Commit message: Ultrasonic Integration

File: src/robot_description/urdf/robot.urdf.xacro (robot description, xacro)
@@ -10,4 +10,7 @@
   <material name="White">
     <color rgba="1 1 1 1"/>
+  </material>
+  <material name="Red">
+    <color rgba="0.8 0.1 0.1 1"/>
   </material>
   <!-- === PROPERTIES === -->
@@ -94,4 +97,32 @@
     </visual>
   </link>
+  <!-- === Ultrasonic Sensor Links === -->
+<link name="ultrasonic_a_link">
+  <visual>
+    <geometry>
+      <cylinder radius="0.01" length="0.02"/>
+    </geometry>
+    <origin xyz="0 0 0" rpy="0 1.5708 0"/> <!-- sideways orientation -->
+    <material name="Red"/>
+  </visual>
+</link>
+<link name="ultrasonic_b_link">
+  <visual>
+    <geometry>
+      <cylinder radius="0.01" length="0.02"/>
+    </geometry>
+    <origin xyz="0 0 0" rpy="0 1.5708 0"/>
+    <material name="Red"/>
+  </visual>
+</link>
+<link name="ultrasonic_c_link">
+  <visual>
+    <geometry>
+      <cylinder radius="0.01" length="0.02"/>
+    </geometry>
+    <origin xyz="0 0 0" rpy="0 1.5708 0"/>
+    <material name="Red"/>
+  </visual>
+</link>
   <!-- === JOINTS === -->
   <joint name="wheel_left_joint" type="continuous">
@@ -122,4 +153,20 @@
     <origin xyz="${camera_xyz}" rpy="${camera_rpy}"/>
   </joint>
+  <!-- === Ultrasonic Sensor Joints === -->
+  <joint name="ultrasonic_a_joint" type="fixed">
+    <parent link="base_link"/>
+    <child link="ultrasonic_a_link"/>
+    <origin xyz="${base_radius} 0 ${-base_height/2 + 0.02}" rpy="0 0 0"/>
+  </joint>
+  <joint name="ultrasonic_b_joint" type="fixed">
+    <parent link="base_link"/>
+    <child link="ultrasonic_b_link"/>
+    <origin xyz="${base_radius * cos(-0.5236)} ${base_radius * sin(-0.5236)} ${-base_height/2 + 0.02}" rpy="0 0 -0.5236"/>
+  </joint>
+  <joint name="ultrasonic_c_joint" type="fixed">
+    <parent link="base_link"/>
+    <child link="ultrasonic_c_link"/>
+    <origin xyz="${base_radius * cos(0.5236)} ${base_radius * sin(0.5236)} ${-base_height/2 + 0.02}" rpy="0 0 0.5236"/>
+  </joint>
   <!-- === ros2_control === -->
   <ros2_control name="diffbot_system" type="system">

Commit message: 1. AB EB AH fixes to DiffBotSystem.cpp to fix map spin

File: src/robot_description/urdf/robot.urdf.xacro (robot description, xacro)
@@ -33,6 +33,4 @@
   <xacro:property name="lidar_xyz"  value="0 0 ${wheel_radius + 0.55}"/>
   <xacro:property name="lidar_rpy"  value="0 0 0"/>
-  <xacro:property name="camera_xyz" value="0.15 0 ${wheel_radius + 0.5}"/>
-  <xacro:property name="camera_rpy" value="0 0 0"/>
   <!-- === LINKS === -->
   <link name="base_link">
@@ -84,14 +82,5 @@
         <cylinder radius="0.05" length="0.03"/>
       </geometry>
-      <origin xyz="0 0 0" rpy="0 0 0"/>
-      <material name="White"/>
-    </visual>
-  </link>
-  <link name="camera_link">
-    <visual>
-      <geometry>
-        <box size="0.05 0.05 0.05"/>
-      </geometry>
-      <origin xyz="0 0 0" rpy="0 0 0"/>
+      <origin xyz="0 0 ${wheel_radius + 0.55}" rpy="0 0 0"/>
       <material name="White"/>
     </visual>
@@ -148,9 +137,4 @@
     <origin xyz="${lidar_xyz}" rpy="${lidar_rpy}"/>
   </joint>
-  <joint name="camera_joint" type="fixed">
-    <parent link="base_link"/>
-    <child  link="camera_link"/>
-    <origin xyz="${camera_xyz}" rpy="${camera_rpy}"/>
-  </joint>
   <!-- === Ultrasonic Sensor Joints === -->
   <joint name="ultrasonic_a_joint" type="fixed">

Commit message: continuing debug of rviz lidar and map drift

File: src/robot_description/urdf/robot.urdf.xacro (robot description, xacro)
@@ -31,5 +31,5 @@
   <xacro:property name="imu_xyz"    value="0 0 ${wheel_radius + 0.01}"/>
   <xacro:property name="imu_rpy"    value="0 0 3.14159"/>
-  <xacro:property name="lidar_xyz"  value="0 0 ${wheel_radius + 0.55}"/>
+  <xacro:property name="lidar_xyz"  value="0 0 .55"/>
   <xacro:property name="lidar_rpy"  value="0 0 0"/>
   <!-- === LINKS === -->
@@ -82,5 +82,5 @@
         <cylinder radius="0.05" length="0.03"/>
       </geometry>
-      <origin xyz="0 0 ${wheel_radius + 0.55}" rpy="0 0 0"/>
+      <origin xyz="0 0 0.55" rpy="0 0 0"/>
       <material name="White"/>
     </visual>

Commit message: 1. AB changed lidar_link to laser_frame to match sllidar_node in control_launch.py and urdf to resolve issue 2. AB changed mapper_params_online_async.yaml to use max scan range of 12 to match lidar specs 3. AB changed bond timeout to 12s in attempt to fix bond timeout issue Tried bond timeout values of 8, 10 and 12 seconds but still getting bond timeout errors for slam_toolbox

File: src/robot_description/urdf/robot.urdf.xacro (robot description, xacro)
@@ -77,5 +77,5 @@
     </visual>
   </link>
-  <link name="lidar_link">
+  <link name="laser_frame">
     <visual>
       <geometry>
@@ -134,5 +134,5 @@
   <joint name="lidar_joint" type="fixed">
     <parent link="base_link"/>
-    <child  link="lidar_link"/>
+    <child  link="laser_frame"/>
     <origin xyz="${lidar_xyz}" rpy="${lidar_rpy}"/>
   </joint>

Commit message: 1. AB a bunch of changes to debug tf issue... it will work

File: src/robot_description/urdf/robot.urdf.xacro (robot description, xacro)
@@ -16,7 +16,7 @@
   <!-- === PROPERTIES === -->
   <!-- Wheels -->
-  <xacro:property name="wheel_radius"       value="0.0325"/>
-  <xacro:property name="wheel_separation"   value="0.292"/>
-  <xacro:property name="wheel_width"        value="0.027"/>
+  <xacro:property name="wheel_radius"       value="0.03329"/> <!-- double-checked 5/16 -AH -->
+  <xacro:property name="wheel_separation"   value="0.294"/> <!-- double-checked 5/16 -AH -->
+  <xacro:property name="wheel_width"        value="0.02528"/> <!-- double-checked 5/16 -AH -->
   <xacro:property name="wheel_mass"         value="0.034"/>
   <xacro:property name="wheel_inertia"      value="${0.5 * wheel_mass * wheel_radius * wheel_radius}"/>
@@ -34,4 +34,13 @@
   <xacro:property name="lidar_rpy"  value="0 0 0"/>
   <!-- === LINKS === -->
+  <!-- <link name="base_footprint">
+    <visual>
+      <geometry>
+        <cylinder radius="${base_radius}" length="${base_height}"/>
+      </geometry>
+      <origin xyz="0 0 0" rpy="0 0 0"/>
+      <material name="Green"/>
+    </visual>
+  </link> -->
   <link name="base_link">
     <inertial>
@@ -115,8 +124,13 @@
 </link>
   <!-- === JOINTS === -->
+<!-- <joint name="base_footprint_to_base_link" type="fixed">
+    <parent link="base_footprint"/>
+    <child  link="base_link"/>
+    <origin xyz="0 0 ${base_height/2.0}" rpy="0 0 0"/>
+</joint> -->
   <joint name="wheel_left_joint" type="continuous">
     <parent link="base_link"/>
     <child  link="wheel_left_link"/>
-    <origin xyz="0 ${-wheel_separation/2.0} 0" rpy="0 0 0"/>
+    <origin xyz="0 ${wheel_separation/2.0} 0" rpy="0 0 0"/>
     <axis xyz="0 1 0"/>
   </joint>
@@ -124,5 +138,5 @@
     <parent link="base_link"/>
     <child  link="wheel_right_link"/>
-    <origin xyz="0 ${wheel_separation/2.0} 0" rpy="0 0 0"/>
+    <origin xyz="0 ${-wheel_separation/2.0} 0" rpy="0 0 0"/>
     <axis xyz="0 1 0"/>
   </joint>

Commit message: More fudge factors, almost there

File: src/robot_description/urdf/robot.urdf.xacro (robot description, xacro)
@@ -132,5 +132,5 @@
     <parent link="base_link"/>
     <child  link="wheel_left_link"/>
-    <origin xyz="0 ${wheel_separation/2.0} 0" rpy="0 0 0"/>
+    <origin xyz="0 ${-wheel_separation/2.0} 0" rpy="0 0 0"/>
     <axis xyz="0 1 0"/>
   </joint>
@@ -138,5 +138,5 @@
     <parent link="base_link"/>
     <child  link="wheel_right_link"/>
-    <origin xyz="0 ${-wheel_separation/2.0} 0" rpy="0 0 0"/>
+    <origin xyz="0 ${wheel_separation/2.0} 0" rpy="0 0 0"/>
     <axis xyz="0 1 0"/>
   </joint>
